Commit message: Revision of Hip axis direction(-x->x) in model file(sdf & urdf) and Applying Control law of "PD + Gravity Compensation"

File: PONGBOT_Q_V2/urdf/PONGBOT_Q_V2.urdf (robot description, URDF)
Before this commit: robot PONGBOT_Q_V2, 14 links, 13 joints
Joints:
- joint FL_HIP_JOINT: axis -1 0 0 -> 1 0 0
- joint FR_HIP_JOINT: axis -1 0 0 -> 1 0 0
- joint RL_HIP_JOINT: axis -1 0 0 -> 1 0 0
- joint RR_HIP_JOINT: axis -1 0 0 -> 1 0 0
