Commit message: Some modes(Trotting, up down, raise leg, jumpping) were added in the CRobot.cpp and there were some corrections of material property in the urdf file because of the Pongbot's parallel link.

File: PONGBOT_Q_V2/urdf/PONGBOT_Q_V2 (copy).urdf (robot description, URDF)
Before this commit: robot PONGBOT_Q_V2, 14 links, 13 joints
Links:
- link FL_THIGH: mass 2.1516 -> 1.8748
- link FR_THIGH: mass 2.1516 -> 1.8748
- link RL_THIGH: mass 2.1516 -> 1.8748
- link RR_THIGH: mass 2.1516 -> 1.8748
