Commit message: Code was merged with HS.

File: pongbot_rviz/urdf/PONGBOT_Q_V2.urdf (robot description, URDF)
Before this commit: robot PONGBOT_Q_V2, 14 links, 13 joints
Links:
- added link FL_TIP, mass 0.01; collision mesh filename=package://pongbot_rviz/meshes/FL_TIP.STL; visual mesh filename=package://pongbot_rviz/meshes/FL_TIP.STL
- added link FR_TIP, mass 0.01; collision mesh filename=package://pongbot_rviz/meshes/FR_TIP.STL; visual mesh filename=package://pongbot_rviz/meshes/FR_TIP.STL
- added link RL_TIP, mass 0.01; collision mesh filename=package://pongbot_rviz/meshes/RL_TIP.STL; visual mesh filename=package://pongbot_rviz/meshes/RL_TIP.STL
- added link RR_TIP, mass 0.01; collision mesh filename=package://pongbot_rviz/meshes/RR_TIP.STL; visual mesh filename=package://pongbot_rviz/meshes/RR_TIP.STL
Joints:
- added joint FL_TIP_JOINT: type fixed, parent FL_CALF, child FL_TIP, origin xyz=-0.015 -0.0004 -0.288 rpy=0 0.7854 0, axis 0 1 0
- added joint FR_TIP_JOINT: type fixed, parent FR_CALF, child FR_TIP, origin xyz=-0.015 -0.0004 -0.288 rpy=0 0.7854 0, axis 0 1 0
- added joint RL_TIP_JOINT: type fixed, parent RL_CALF, child RL_TIP, origin xyz=0.015 0.001 -0.288 rpy=0 5.497 0, axis 0 1 0
- added joint RR_TIP_JOINT: type fixed, parent RR_CALF, child RR_TIP, origin xyz=0.015 0.001 -0.288 rpy=0 5.497 0, axis 0 1 0
