Commit message: Fast trot walking motion was generated.

File: model/PONGBOT_Q_V4/urdf/PONGBOT_Q_V4.urdf (robot description, URDF)
Before this commit: robot PONGBOT_Q_V4, 18 links, 17 joints
Links:
- removed link FL_TIP
- removed link FR_TIP
- removed link RL_TIP
- removed link RR_TIP
Joints:
- removed joint FL_TIP_JOINT
- removed joint FR_TIP_JOINT
- removed joint RL_TIP_JOINT
- removed joint RR_TIP_JOINT
